File: UINIO-MCU-GD32F350RBT6.kicad_sch (KiCad schematic)
At the start: 1 part

Commit message: Initializing the project
Parts:
- added C? (x2): 1uF, Capacitor_SMD:C_0402_1005Metric, symbol Device:C
- added D?: LED_Red, LED_SMD:LED_0603_1608Metric, symbol Device:LED
- added J? (x2): Conn_01x32_Male, symbol Connector:Conn_01x32_Male
- added J?: Conn_01x05_Male, symbol Connector:Conn_01x05_Male
- added R?: 2K, Resistor_SMD:R_0402_1005Metric, symbol Device:R
- added SW?: 下载按键, Uinio:KEY-SMD_4P-L4.2-W3.4-P2.15-LS4.7, symbol Uinio:Key_YTS_A016S_1
- added SW?: 复位按键, Uinio:KEY-SMD_4P-L4.2-W3.4-P2.15-LS4.7, symbol Uinio:Key_YTS_A016S_1
- added U?: ME6211C33M5G-N, Uinio:SOT-23-5_L3.0-W1.7-P0.95-LS2.8-BR, symbol Uinio:ME6211
- added USB?: USB_Type_C_16Pin, Uinio:USB-C-SMD_TYPEC-304J-BCP16, symbol Uinio:USB_Type_C_16Pin
Connections:
- new net: D?.2 (A), R?.1
- new net GND: C?.1, C?.1, D?.1 (K), U?.2 (Vss), USB?.13 (GND), USB?.14 (GND), USB?.15 (GND), USB?.16 (GND), USB?.A1B12 (GND), USB?.B1A12 (GND)
- new net USB_Data+: USB?.A6 (DP1), USB?.B6 (DP2)
- new net USB_Data-: USB?.A7 (DN1), USB?.B7 (DN2)
- new net VDD_3.3V: C?.2, U?.5 (Vout)
- new net VDD_5V: C?.2, R?.2, U?.1 (Vin), U?.3 (CE), USB?.A4B9 (VBUS), USB?.B4A9 (VBUS)
- no-connect marks 0 -> 5
Other:
- note added: "3.3V 线性稳压电路"
- note added: "USB Type-C 接口电路"
- moved on the sheet: U?

Commit message: Initializing the project.
Parts:
- added C? (x2): 0.1uF, symbol Device:C
- added C? (x4): C, symbol Device:C
- added R?: 1M, symbol Device:R
- added Y?: 8MHz, Crystal:Crystal_SMD_3225-4Pin_3.2x2.5mm, symbol Device:Crystal_GND24
- added Y?: 32.768 KHz, Uinio:CRYSTAL-FC135-32.768, symbol Uinio:FC135-32.768
Connections:
- net GND: now also U?.31 (VSS), U?.63 (VSS), C?.1, C?.1, C?.1, C?.1, C?.1, C?.1
- net VDD_3.3V: now also U?.32 (VDD), U?.64 (VDD), C?.2, C?.2
- net VBAT: now reaches U?.1 (VBAT)
- net PC2: now reaches U?.10 (PC2)
- net PC3: now reaches U?.11 (PC3)
- net VSSA: now reaches U?.12 (VSSA)
- net VDDA: now reaches U?.13 (VDDA)
- net PA0: now reaches U?.14 (PA0)
- net PA1: now reaches U?.15 (PA1)
- net PA2: now reaches U?.16 (PA2)
- net PA3: now reaches U?.17 (PA3)
- net PF4: now reaches U?.18 (PF4)
- net PF5: now reaches U?.19 (PF5)
- net PC13: now reaches U?.2 (PC13)
- net PA4: now reaches U?.20 (PA4)
- net PA5: now reaches U?.21 (PA5)
- net PA6: now reaches U?.22 (PA6)
- net PA7: now reaches U?.23 (PA7)
- net PC4: now reaches U?.24 (PC4)
- net PC5: now reaches U?.25 (PC5)
- net PB0: now reaches U?.26 (PB0)
- net PB1: now reaches U?.27 (PB1)
- net PB2: now reaches U?.28 (PB2)
- net PB10: now reaches U?.29 (PB10)
- net at U?.3 (PC14-OSC32IN): now also C?.2, Y?.1
- net PB11: now reaches U?.30 (PB11)
- net PB12: now reaches U?.33 (PB12)
- net PB13: now reaches U?.34 (PB13)
- net PB14: now reaches U?.35 (PB14)
- net PB15: now reaches U?.36 (PB15)
- net PC6: now reaches U?.37 (PC6)
- net PC7: now reaches U?.38 (PC7)
- net PC8: now reaches U?.39 (PC8)
- net at U?.4 (PC15-OSC32OUT): now also C?.2, Y?.2 (GND)
- net PC9: now reaches U?.40 (PC9)
- net PA8: now reaches U?.41 (PA8)
- net PA9: now reaches U?.42 (PA9)
- net PA10: now reaches U?.43 (PA10)
- net PA11: now reaches U?.44 (PA11)
- net PA12: now reaches U?.45 (PA12)
- net PA13: now reaches U?.46 (PA13)
- net PF6: now reaches U?.47 (PF6)
- net PF7: now reaches U?.48 (PF7)
- net PA14: now reaches U?.49 (PA14)
- net PF0: now reaches U?.5 (PF0-OSCIN)
- net PF0: now also R?.1, Y?.3
- net PA15: now reaches U?.50 (PA15)
- net PC10: now reaches U?.51 (PC10)
- net PC11: now reaches U?.52 (PC11)
- net PC12: now reaches U?.53 (PC12)
- net PD2: now reaches U?.54 (PD2)
- net PB3: now reaches U?.55 (PB3)
- net PB4: now reaches U?.56 (PB4)
- net PB5: now reaches U?.57 (PB5)
- net PB6: now reaches U?.58 (PB6)
- net PB7: now reaches U?.59 (PB7)
- net PF1: now reaches U?.6 (PF1-OSCOUT)
- net PF1: now also R?.2, Y?.1
- net BOOT0: now reaches U?.60 (BOOT0)
- net PB8: now reaches U?.61 (PB8)
- net PB9: now reaches U?.62 (PB9)
- net NRST: now reaches U?.7 (NRST)
- net PC0: now reaches U?.8 (PC0)
- net PC1: now reaches U?.9 (PC1)
- new net: C?.2, Y?.4
- new net: C?.2, Y?.2
Other:
- moved on the sheet: SW?

Commit message: Update schematic diagram.
Parts:
- removed SW?: 下载按键, Uinio:KEY-SMD_4P-L4.2-W3.4-P2.15-LS4.7, symbol Uinio:Key_YTS_A016S_1
- added C? (x2): 0.1uF, symbol Device:C
- added L?: 1KΩ 100Mhz, symbol Device:L
- added R? (x2): 10K, symbol Device:R
- added R?: 0R, symbol Device:R
- added SW?: BOOT0, Uinio:KEY-SMD_4P-L4.2-W3.4-P2.15-LS4.7, symbol Uinio:Key_YTS_A016S_1
- C? (x2): value C -> 10pF
- C? (x2): value C -> 20pF
- SW?: value 复位按键 -> NRST
Connections:
- net BOOT0: now also J?.5 (Pin_5); no longer U?.60 (BOOT0)
- net GND: now also J?.13 (Pin_13), J?.2 (Pin_2), J?.3 (Pin_3), J?.32 (Pin_32), J?.4 (Pin_4), J?.6 (Pin_6), SW?.3, SW?.4, C?.1, C?.2, R?.2, R?.2, SW?.1, SW?.2
- net NRST: now also J?.7 (Pin_7), SW?.1, SW?.2, C?.1, R?.2
- net PA0: now also J?.14 (Pin_14)
- net PA1: now also J?.15 (Pin_15)
- net PA10: now also J?.22 (Pin_22)
- net PA11: now also J?.21 (Pin_21)
- net PA12: now also J?.20 (Pin_20)
- net PA13: now also J?.19 (Pin_19)
- net PA14: now also J?.16 (Pin_16)
- net PA15: now also J?.15 (Pin_15)
- net PA2: now also J?.16 (Pin_16)
- net PA3: now also J?.17 (Pin_17)
- net PA4: now also J?.20 (Pin_20)
- net PA5: now also J?.21 (Pin_21)
- net PA6: now also J?.22 (Pin_22)
- net PA7: now also J?.23 (Pin_23)
- net PA8: now also J?.24 (Pin_24)
- net PA9: now also J?.23 (Pin_23)
- net PB0: now also J?.26 (Pin_26)
- net PB1: now also J?.27 (Pin_27)
- net PB10: now also J?.29 (Pin_29)
- net PB11: now also J?.30 (Pin_30)
- net PB12: now also J?.32 (Pin_32)
- net PB13: now also J?.31 (Pin_31)
- net PB14: now also J?.30 (Pin_30)
- net PB15: now also J?.29 (Pin_29)
- net PB2: now also J?.28 (Pin_28)
- net PB3: now also J?.10 (Pin_10)
- net PB4: now also J?.9 (Pin_9)
- net PB5: now also J?.8 (Pin_8)
- net PB6: now also J?.7 (Pin_7)
- net PB7: now also J?.6 (Pin_6)
- net PB8: now also J?.4 (Pin_4)
- net PB9: now also J?.3 (Pin_3)
- net PC0: now also J?.8 (Pin_8)
- net PC1: now also J?.9 (Pin_9)
- net PC10: now also J?.14 (Pin_14)
- net PC11: now also J?.13 (Pin_13)
- net PC12: now also J?.12 (Pin_12)
- net PC13: now also J?.2 (Pin_2)
- net PC2: now also J?.10 (Pin_10)
- net PC3: now also J?.11 (Pin_11)
- net PC4: now also J?.24 (Pin_24)
- net PC5: now also J?.25 (Pin_25)
- net PC6: now also J?.28 (Pin_28)
- net PC7: now also J?.27 (Pin_27)
- net PC8: now also J?.26 (Pin_26)
- net PC9: now also J?.25 (Pin_25)
- net PD2: now also J?.11 (Pin_11)
- net PF4: now also J?.18 (Pin_18)
- net PF5: now also J?.19 (Pin_19)
- net PF6: now also J?.18 (Pin_18)
- net PF7: now also J?.17 (Pin_17)
- net VBAT: now also J?.1 (Pin_1)
- net VDDA: now also L?.2
- net VDD_3.3V: now also J?.1 (Pin_1), J?.1 (Pin_1), J?.12 (Pin_12), J?.4 (Pin_4), J?.5 (Pin_5), L?.1, R?.1, SW?.3, SW?.4
- net VDD_5V: now also J?.31 (Pin_31)
- net VSSA: now also R?.1
- net SWDIO: now reaches J?.2 (Pin_2)
- net SWCLK: now reaches J?.3 (Pin_3)
- net RESET: now reaches J?.5 (Pin_5)
- new net: C?.2, R?.1, U?.60 (BOOT0)
Other:
- moved on the sheet: C?, D?, J?, R?, SW?, U?, USB?, Y?

Commit message: Finish PCB layout.
Parts:
- removed J?: Conn_01x05_Male, symbol Connector:Conn_01x05_Male
- removed R?: 0R, symbol Device:R
- removed Y?: 32.768 KHz, Uinio:CRYSTAL-FC135-32.768, symbol Uinio:FC135-32.768
- added J3: Conn_01x04_Male, Connector_PinHeader_2.54mm:PinHeader_1x04_P2.54mm_Vertical, symbol Connector:Conn_01x04_Male
- added R5, R6: 10K, Resistor_SMD:R_0603_1608Metric, symbol Device:R
- added R7, R8: 50R, Resistor_SMD:R_0603_1608Metric, symbol Device:R
- added R9: 1.5K, Resistor_SMD:R_0603_1608Metric, symbol Device:R
- added Y1: 32.768KHz, Uinio:CRYSTAL-FC135-32.768, symbol Uinio:Crystal-32.768KHz
- C1, C3: renamed from C?; footprint Capacitor_SMD:C_0402_1005Metric -> Capacitor_SMD:C_0603_1608Metric
- C10, C2, C4, C5, C6, C7, C8, C9: renamed from C?; footprint (none) -> Capacitor_SMD:C_0603_1608Metric
- J1, J2: renamed from J?; footprint (none) -> Connector_PinHeader_2.54mm:PinHeader_1x32_P2.54mm_Vertical
- L1: renamed from L?; footprint (none) -> Inductor_SMD:L_0603_1608Metric
- R1: renamed from R?; footprint Resistor_SMD:R_0402_1005Metric -> Resistor_SMD:R_0603_1608Metric
- R2, R3, R4: renamed from R?; footprint (none) -> Resistor_SMD:R_0603_1608Metric
- gave numbers to parts that had none: 7
Connections:
- net BOOT0: now also C2.2, R2.1, U2.60 (BOOT0)
- net GND: now also L1.1, J3.1 (Pin_1), R5.1
- net PA11: now also R8.1
- net PA12: now also R7.1, R9.2
- net USB_Data+: now also R7.2
- net USB_Data-: now also R8.2
- net VDD_3.3V: now also U2.13 (VDDA), J3.4 (Pin_4), R6.2, R9.1; no longer L1.1
- net VSSA: now also L1.2
- net at C8.2, U2.3 (PC14-OSC32IN): now also Y1.2 (GND)
- net at C9.2, U2.4 (PC15-OSC32OUT): now also Y1.1
- net PA13 renamed PA13/SWDIO
- net PA13/SWDIO: now also J3.3 (Pin_3), R6.1
- net PA14 renamed PA14/SWCLK
- net PA14/SWCLK: now also J3.2 (Pin_2), R5.2
- removed net VDDA: L1.2, U2.13 (VDDA)
Other:
- note added: "32Pin 2.54mm 排针"
- note added: "GD32F350RBT6 最小系统"
- note added: "SWD 调试接口"
- moved on the sheet: C1, C10, C2, C3, C4, C5, C6, C7, C8, C9, D1, J1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

Commit message: Finish PCB layout.
Connections:
- net GND: now also J1.5 (Pin_5); no longer J1.6 (Pin_6)
- net VDD_3.3V: now also J1.31 (Pin_31), J1.6 (Pin_6); no longer J1.4 (Pin_4), J1.5 (Pin_5)
- net VDD_5V: now also J1.4 (Pin_4); no longer J1.31 (Pin_31)
Changed lines of the file:
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@@
     (stroke (width 0) (type default) (color 0 0 0 0))
   )
-  (wire (pts (xy 45.72 40.64) (xy 36.83 40.64))
+  (wire (pts (xy 45.72 38.1) (xy 36.83 38.1))
     (stroke (width 0) (type default) (color 0 0 0 0))
   )
@@
     (effects (font (size 1.27 1.27)) (justify right bottom))
   )
-  (label "VDD_5V" (at 45.72 104.14 180)
+  (label "VDD_5V" (at 45.72 35.56 180)
     (effects (font (size 1.27 1.27)) (justify right bottom))
   )
@@
     (effects (font (size 1.27 1.27)) (justify left bottom))
   )
-  (label "VDD_3.3V" (at 45.72 38.1 180)
+  (label "VDD_3.3V" (at 45.72 104.14 180)
     (effects (font (size 1.27 1.27)) (justify right bottom))
   )
@@
     (effects (font (size 1.27 1.27)) (justify right bottom))
   )
-  (label "VDD_3.3V" (at 45.72 35.56 180)
+  (label "VDD_3.3V" (at 45.72 40.64 180)
     (effects (font (size 1.27 1.27)) (justify right bottom))
   )
@@
     (pin "1")
   )
-  (symbol (lib_id "power:GND") (at 36.83 40.64 270) (unit 1)
-    (in_bom yes) (on_board yes)
-    (property "Reference" "#PWR04" (id 0) (at 30.48 40.64 0)
-      (effects (font (size 1.27 1.27)) hide)
-    )
-    (property "Value" "GND" (id 1) (at 33.02 40.6401 90)
-      (effects (font (size 1.27 1.27)) (justify right))
-    )
-    (property "Footprint" "" (id 2) (at 36.83 40.64 0)
-      (effects (font (size 1.27 1.27)) hide)
-    )
-    (property "Datasheet" "" (id 3) (at 36.83 40.64 0)
-      (effects (font (size 1.27 1.27)) hide)
-    )
+  (symbol (lib_id "power:GND") (at 36.83 38.1 270) (unit 1)
+    (in_bom yes) (on_board yes)
+    (property "Reference" "#PWR04" (id 0) (at 30.48 38.1 0)
+      (effects (font (size 1.27 1.27)) hide)
+    )
+    (property "Value" "GND" (id 1) (at 33.02 38.1001 90)
+      (effects (font (size 1.27 1.27)) (justify right))
+    )
+    (property "Footprint" "" (id 2) (at 36.83 38.1 0)
+      (effects (font (size 1.27 1.27)) hide)
+    )
+    (property "Datasheet" "" (id 3) (at 36.83 38.1 0)
+      (effects (font (size 1.27 1.27)) hide)
+    )

Commit message: Release UINIO-MCU-GD32F350RBT6 version 1.0.0.
Parts:
- J3: footprint Connector_PinHeader_2.54mm:PinHeader_1x04_P2.54mm_Vertical -> Connector_PinHeader_2.54mm:PinHeader_1x04_P2.54mm_Horizontal
Other:
- moved on the sheet: C1, C3, J1, J2, U1

Commit message: Release UINIO-MCU-GD32F350RBT6 version 1.0.0.
Parts:
- J3: footprint Connector_PinHeader_2.54mm:PinHeader_1x04_P2.54mm_Horizontal -> Connector_PinHeader_2.54mm:PinHeader_1x04_P2.54mm_Vertical
Connections:
- net GND: now also J1.1 (Pin_1), J2.1 (Pin_1); no longer J1.5 (Pin_5), J2.2 (Pin_2)
- net PC13: now also J1.6 (Pin_6); no longer J1.2 (Pin_2)
- net VBAT: now also J1.5 (Pin_5); no longer J1.1 (Pin_1)
- net VDD_3.3V: now also J1.4 (Pin_4), J2.2 (Pin_2); no longer J1.6 (Pin_6), J2.1 (Pin_1)
- net VDD_5V: now also J1.2 (Pin_2); no longer J1.4 (Pin_4)
Changed lines of the file:
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@@
     (stroke (width 0) (type default) (color 0 0 0 0))
   )
-  (wire (pts (xy 78.74 30.48) (xy 87.63 30.48))
+  (wire (pts (xy 78.74 27.94) (xy 87.63 27.94))
     (stroke (width 0) (type default) (color 0 0 0 0))
   )
@@
     (stroke (width 0) (type default) (color 0 0 0 0))
   )
-  (wire (pts (xy 46.355 33.02) (xy 37.465 33.02))
+  (wire (pts (xy 46.355 27.94) (xy 37.465 27.94))
     (stroke (width 0) (type default) (color 0 0 0 0))
   )
@@
     (stroke (width 0) (type default) (color 0 0 0 0))
   )
-  (wire (pts (xy 46.355 38.1) (xy 37.465 38.1))
+  (wire (pts (xy 46.355 33.02) (xy 37.465 33.02))
     (stroke (width 0) (type default) (color 0 0 0 0))
   )
@@
     (effects (font (size 1.27 1.27)) (justify right bottom))
   )
-  (label "VDD_5V" (at 46.355 35.56 180)
+  (label "VDD_5V" (at 46.355 30.48 180)
     (effects (font (size 1.27 1.27)) (justify right bottom))
   )
@@
     (effects (font (size 1.27 1.27)) (justify right bottom))
   )
-  (label "VDD_3.3V" (at 46.355 40.64 180)
+  (label "VDD_3.3V" (at 46.355 35.56 180)
     (effects (font (size 1.27 1.27)) (justify right bottom))
   )
@@
     (effects (font (size 1.27 1.27)) (justify left bottom))
   )
-  (label "VBAT" (at 46.355 27.94 180)
+  (label "VBAT" (at 46.355 38.1 180)
     (effects (font (size 1.27 1.27)) (justify right bottom))
   )
@@
     (effects (font (size 1.27 1.27)) (justify right bottom))
   )
-  (label "VDD_3.3V" (at 78.74 27.94 0)
+  (label "VDD_3.3V" (at 78.74 30.48 0)
     (effects (font (size 1.27 1.27)) (justify left bottom))
   )
@@
     (effects (font (size 1.27 1.27)) (justify left bottom))
   )
-  (label "PC13" (at 46.355 30.48 180)
+  (label "PC13" (at 46.355 40.64 180)
     (effects (font (size 1.27 1.27)) (justify right bottom))
   )
@@
     (pin "4")
   )
-  (symbol (lib_id "power:GND") (at 37.465 33.02 270) (unit 1)
-    (in_bom yes) (on_board yes)
-    (property "Reference" "#PWR03" (id 0) (at 31.115 33.02 0)
-      (effects (font (size 1.27 1.27)) hide)
-    )
-    (property "Value" "GND" (id 1) (at 33.655 33.0201 90)
-      (effects (font (size 1.27 1.27)) (justify right))
-    )
-    (property "Footprint" "" (id 2) (at 37.465 33.02 0)
-      (effects (font (size 1.27 1.27)) hide)
-    )
-    (property "Datasheet" "" (id 3) (at 37.465 33.02 0)
+  (symbol (lib_id "power:GND") (at 37.465 27.94 270) (unit 1)
+    (in_bom yes) (on_board yes)
+    (property "Reference" "#PWR03" (id 0) (at 31.115 27.94 0)
+      (effects (font (size 1.27 1.27)) hide)
+    )
+    (property "Value" "GND" (id 1) (at 33.655 27.9401 90)
+      (effects (font (size 1.27 1.27)) (justify right))
+    )
+    (property "Footprint" "" (id 2) (at 37.465 27.94 0)
+      (effects (font (size 1.27 1.27)) hide)
+    )
+    (property "Datasheet" "" (id 3) (at 37.465 27.94 0)
       (effects (font (size 1.27 1.27)) hide)
     )
@@
     (pin "2")
   )
-  (symbol (lib_id "power:GND") (at 87.63 30.48 90) (unit 1)
-    (in_bom yes) (on_board yes)
-    (property "Reference" "#PWR08" (id 0) (at 93.98 30.48 0)
-      (effects (font (size 1.27 1.27)) hide)
-    )
-    (property "Value" "GND" (id 1) (at 91.44 30.4799 90)
-      (effects (font (size 1.27 1.27)) (justify right))
-    )
-    (property "Footprint" "" (id 2) (at 87.63 30.48 0)
-      (effects (font (size 1.27 1.27)) hide)
-    )
-    (property "Datasheet" "" (id 3) (at 87.63 30.48 0)
+  (symbol (lib_id "power:GND") (at 87.63 27.94 90) (unit 1)
+    (in_bom yes) (on_board yes)
+    (property "Reference" "#PWR08" (id 0) (at 93.98 27.94 0)
+      (effects (font (size 1.27 1.27)) hide)
+    )
+    (property "Value" "GND" (id 1) (at 91.44 27.9399 90)
+      (effects (font (size 1.27 1.27)) (justify right))
+    )
+    (property "Footprint" "" (id 2) (at 87.63 27.94 0)
+      (effects (font (size 1.27 1.27)) hide)
+    )
+    (property "Datasheet" "" (id 3) (at 87.63 27.94 0)
       (effects (font (size 1.27 1.27)) hide)
     )
@@
     (property "Reference" "J3" (id 0) (at 215.9 135.89 0))
     (property "Value" "Conn_01x04_Male" (id 1) (at 217.17 151.13 0))
-    (property "Footprint" "Connector_PinHeader_2.54mm:PinHeader_1x04_P2.54mm_Horizontal" (id 2) (at 213.36 142.24 0)
+    (property "Footprint" "Connector_PinHeader_2.54mm:PinHeader_1x04_P2.54mm_Vertical" (id 2) (at 213.36 142.24 0)
       (effects (font (size 1.27 1.27)) hide)
     )
@@
     (pin "1")
   )
-  (symbol (lib_id "power:GND") (at 37.465 38.1 270) (unit 1)
-    (in_bom yes) (on_board yes)
-    (property "Reference" "#PWR04" (id 0) (at 31.115 38.1 0)
-      (effects (font (size 1.27 1.27)) hide)
-    )
-    (property "Value" "GND" (id 1) (at 33.655 38.1001 90)
-      (effects (font (size 1.27 1.27)) (justify right))
-    )
-    (property "Footprint" "" (id 2) (at 37.465 38.1 0)
-      (effects (font (size 1.27 1.27)) hide)
-    )
-    (property "Datasheet" "" (id 3) (at 37.465 38.1 0)
+  (symbol (lib_id "power:GND") (at 37.465 33.02 270) (unit 1)
+    (in_bom yes) (on_board yes)
+    (property "Reference" "#PWR04" (id 0) (at 31.115 33.02 0)
+      (effects (font (size 1.27 1.27)) hide)
+    )
+    (property "Value" "GND" (id 1) (at 33.655 33.0201 90)
+      (effects (font (size 1.27 1.27)) (justify right))
+    )
+    (property "Footprint" "" (id 2) (at 37.465 33.02 0)
+      (effects (font (size 1.27 1.27)) hide)
+    )
+    (property "Datasheet" "" (id 3) (at 37.465 33.02 0)
       (effects (font (size 1.27 1.27)) hide)
     )
@@
     )
     (path "/7de278ff-98fe-4376-acd3-f3de0c1b8a8a"
-      (reference "J3") (unit 1) (value "Conn_01x04_Male") (footprint "Connector_PinHeader_2.54mm:PinHeader_1x04_P2.54mm_Horizontal")
+      (reference "J3") (unit 1) (value "Conn_01x04_Male") (footprint "Connector_PinHeader_2.54mm:PinHeader_1x04_P2.54mm_Vertical")
     )
     (path "/29857437-9f6a-44af-9940-c4d0e4a35c6f"

Commit message: Upgrade version 2.0.0.
Parts:
- removed J1, J2: Conn_01x32_Male, Connector_PinHeader_2.54mm:PinHeader_1x32_P2.54mm_Vertical, symbol Connector:Conn_01x32_Male
- removed J3: Conn_01x04_Male, Connector_PinHeader_2.54mm:PinHeader_1x04_P2.54mm_Vertical, symbol Connector:Conn_01x04_Male
- added J1, J2: Conn_01x32_Pin, Connector_PinHeader_2.54mm:PinHeader_1x32_P2.54mm_Vertical, symbol Connector:Conn_01x32_Pin
- added J3: Conn_01x04_Pin, Connector_PinHeader_2.54mm:PinHeader_1x04_P2.54mm_Vertical, symbol Connector:Conn_01x04_Pin
Connections:
- net BOOT0: now also J2.5 (Pin_5)
- net GND: now also J1.1 (Pin_1), J1.13 (Pin_13), J1.3 (Pin_3), J1.32 (Pin_32), J2.1 (Pin_1), J3.1 (Pin_1)
- net NRST: now also J1.7 (Pin_7)
- net PA0: now also J1.14 (Pin_14)
- net PA1: now also J1.15 (Pin_15)
- net PA10: now also J2.22 (Pin_22)
- net PA11: now also J2.21 (Pin_21)
- net PA12: now also J2.20 (Pin_20)
- net PA13/SWDIO: now also J2.19 (Pin_19), J3.3 (Pin_3)
- net PA14/SWCLK: now also J2.16 (Pin_16), J3.2 (Pin_2)
- net PA15: now also J2.15 (Pin_15)
- net PA2: now also J1.16 (Pin_16)
- net PA3: now also J1.17 (Pin_17)
- net PA4: now also J1.20 (Pin_20)
- net PA5: now also J1.21 (Pin_21)
- net PA6: now also J1.22 (Pin_22)
- net PA7: now also J1.23 (Pin_23)
- net PA8: now also J2.24 (Pin_24)
- net PA9: now also J2.23 (Pin_23)
- net PB0: now also J1.26 (Pin_26)
- net PB1: now also J1.27 (Pin_27)
- net PB10: now also J1.29 (Pin_29)
- net PB11: now also J1.30 (Pin_30)
- net PB12: now also J2.32 (Pin_32)
- net PB13: now also J2.31 (Pin_31)
- net PB14: now also J2.30 (Pin_30)
- net PB15: now also J2.29 (Pin_29)
- net PB2: now also J1.28 (Pin_28)
- net PB3: now also J2.10 (Pin_10)
- net PB4: now also J2.9 (Pin_9)
- net PB5: now also J2.8 (Pin_8)
- net PB6: now also J2.7 (Pin_7)
- net PB7: now also J2.6 (Pin_6)
- net PB8: now also J2.4 (Pin_4)
- net PB9: now also J2.3 (Pin_3)
- net PC0: now also J1.8 (Pin_8)
- net PC1: now also J1.9 (Pin_9)
- net PC10: now also J2.14 (Pin_14)
- net PC11: now also J2.13 (Pin_13)
- net PC12: now also J2.12 (Pin_12)
- net PC13: now also J1.6 (Pin_6)
- net PC2: now also J1.10 (Pin_10)
- net PC3: now also J1.11 (Pin_11)
- net PC4: now also J1.24 (Pin_24)
- net PC5: now also J1.25 (Pin_25)
- net PC6: now also J2.28 (Pin_28)
- net PC7: now also J2.27 (Pin_27)
- net PC8: now also J2.26 (Pin_26)
- net PC9: now also J2.25 (Pin_25)
- net PD2: now also J2.11 (Pin_11)
- net PF4: now also J1.18 (Pin_18)
- net PF5: now also J1.19 (Pin_19)
- net PF6: now also J2.18 (Pin_18)
- net PF7: now also J2.17 (Pin_17)
- net VBAT: now also J1.5 (Pin_5)
- net VDD_3.3V: now also J1.12 (Pin_12), J1.31 (Pin_31), J1.4 (Pin_4), J2.2 (Pin_2), J3.4 (Pin_4)
- net VDD_5V: now also J1.2 (Pin_2)
